File: lorapuck.kicad_pcb (KiCad board)
At the start: 4 copper layers, 30 x 43 mm, 49 parts, among them J1 USB_C_Receptacle_USB2.0_16P, SW1 BOOTSEL, SW2 RESET, U1 SX1262IMLTRT, U2 RP2040, U3 W25Q128JVS, U4 PE4259, U5 AP2112K-3.3, Y1 32MHz, Y2 12MHz

Commit message: edited the usbc receptacle and added a weather sensor!
Parts:
- added C26: 100nF, Capacitor_SMD:C_0402_1005Metric, F.Cu at (80.9, 111.8)
- added R10: 4.7k, Resistor_SMD:R_0402_1005Metric, F.Cu at (81.1, 106.4)
- added R9: 4.7k, Resistor_SMD:R_0402_1005Metric, F.Cu at (81.1, 105.4)
- added U6: SHTC3, Sensor_Humidity:Sensirion_DFN-4-1EP_2x2mm_P1mm_EP0.7x1.6mm, F.Cu at (80.7, 109.9)
- moved C25 14.0 mm to (100.1, 91.4), turned to 90 degrees
- moved FB1 12.2 mm to (88.6, 88.9), turned to 0 degrees
- moved U5 11.2 mm to (97.5, 92.0), turned to -90 degrees
- moved J1 8.20 mm to (93.1, 83.4), turned to 180 degrees
- moved R8 8.02 mm to (91.1, 89.4), turned to -90 degrees
- moved C24 4.61 mm to (96.0, 89.0), turned to 0 degrees
- moved R7 4.30 mm to (94.6, 89.4), turned to -90 degrees
- moved C1 1.47 mm to (84.0, 103.5), turned to -90 degrees
Connections:
- U2 pad 2: unconnected-(U2-GPIO0-Pad2) -> /IO0
- U2 pad 3: unconnected-(U2-GPIO1-Pad3) -> /IO1
Routing:
- net VBUS: track 16.8 -> 7.94 mm, vias 2 -> 0
- net Net-(U6-SCL): track 0.00 -> 6.05 mm, vias 0 -> 2
- net /IO1: track 0.00 -> 4.35 mm
- net /IO0: track 0.00 -> 4.10 mm
- net Net-(U6-SDA): track 0.00 -> 3.34 mm
- net /USB_DP: track 19.8 -> 16.9 mm, vias 2 -> 0
- net Earth: track 91.0 -> 93.2 mm, vias 27 -> 29
- net +3V3: track 51.9 -> 53.6 mm
- net /USB_DM: track 17.6 -> 16.8 mm
- net Net-(J1-SHIELD): track 19.9 -> 19.7 mm, vias 1 -> 0
Other:
- outline, holes or cut-outs redrawn
