File: lorapuck.kicad_sch (KiCad schematic)
At the start: 49 parts, among them J1 USB_C_Receptacle_USB2.0_16P, SW1 BOOTSEL, SW2 RESET, U1 SX1262IMLTRT, U2 RP2040, U3 W25Q128JVS, U4 PE4259, U5 AP2112K-3.3, Y1 32MHz, Y2 12MHz

Commit message: edited the usbc receptacle and added a weather sensor!
Parts:
- added C26: 100nF, Capacitor_SMD:C_0402_1005Metric, symbol Device:C
- added R10, R9: 4.7k, Resistor_SMD:R_0402_1005Metric, symbol Device:R_US
- added U6: SHTC3, Sensor_Humidity:Sensirion_DFN-4-1EP_2x2mm_P1mm_EP0.7x1.6mm, symbol Sensor_Humidity:SHTC3
Connections:
- net +3V3: now also C26.2, U6.1 (VDD)
- net Earth: now also C26.1, U6.4 (VSS)
- net IO0: now reaches U2.2 (GPIO0)
- net IO0: now also R9.1
- net IO1: now reaches U2.3 (GPIO1)
- net IO1: now also R10.2
- new net: R10.1, U6.3 (SDA)
- new net: R9.2, U6.2 (SCL)
- no-connect marks 29 -> 27
Other:
- moved on the sheet: C15, C22, C23, R4, R6, SW1, SW2, U3, Y2
